File: KiCAD/jSmartSW.kicad_pcb (KiCad board)
At the start: 2 copper layers, 133.5 x 54.6 mm, 23 parts, among them J1 Audio Out, J2 USB4085-GF-A_REVB, J3 EXT, J4 PJ-002A, J5 SBH11-PBPC-D07-RA-BK, J6 Backfeed Power To USBC, P1 To RT4K, P2 From switch output, U1 PICO, U2 SN74LXC1T14DCKR

Commit message: Update Main PCB Silkscreen
Parts:
- removed R4: 10K, Resistor_SMD:R_0603_1608Metric_Pad0.98x0.95mm_HandSolder
- added D2: SMBJ5343B-TP, Diode_SMD:D_SMB, F.Cu at (91.4, 87.6)
- added G***: LOGO, jSmartSW:QR, B.Cu at (92.3, 110.0)
- added R2: 10K, Resistor_SMD:R_0603_1608Metric_Pad0.98x0.95mm_HandSolder, B.Cu at (153.9, 87.9)
- moved R3 3.69 mm to (150.2, 87.9), turned to 0 degrees
Connections:
- R3 pad 1: Net-(J2-CC1) -> Net-(J2-CC2)
Other:
- board text added: "USB Function"
- board text removed: "Enable USB Function"
